File: carte_tutos/carte_tutos.kicad_pcb (KiCad board)
At the start: 2 copper layers, 133 x 117 mm, 99 parts, among them J1 Conn_01x03_Male, J2 Conn_01x03_Male, J3 Barrel_Jack, J4 Conn_01x04_Male, J5 Conn_01x02_Male, J6 Conn_01x03_Male, J7 Conn_01x02_Male, J8 Conn_01x03_Male, Q1 SFH_3410-Z, SW1 Rotary_Encoder_Switch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

Commit message: WIP? Will be cleaned up!
Parts:
- moved R20 0.13 mm to (98.4, 74.9)
